File: SDEX2M2 MicroSD Express Breakout Board/SDEX2M2 Breakout Board.kicad_pcb (KiCad board)
At the start: 6 copper layers, 35.1 x 31.8 mm, 2 parts, among them J1 SDEX2M2 Breakout, J2 Conn_02x08_Top_Bottom

Commit message: Updated schematic and breakout board
Connections:
- net Net-(J1-PCIe_RX+) renamed /RX+
- net Net-(J1-PCIe_RX-) renamed /RX-
- net Net-(J1-PCIe_TX+) renamed /TX+
- net Net-(J1-PCIe_TX-) renamed /TX-
- net Net-(J1-REFCLK+/DAT0) renamed /REFCLK+
- net Net-(J1-REFCLK-/DAT1) renamed /REFCLK-
Routing:
- net Net-(J1-3V3): track 34.7 -> 31.1 mm, vias 5 -> 3
- net /REFCLK-: track 43.6 -> 44.4 mm
- net /RX-: track 42.1 -> 42.6 mm
